File: HARDWARE/NG3ControllerBoard.sch (EAGLE design)
At the start: 10 parts, among them U1 ATMEGA328P-AU, Y1 RESONATORSMD

Commit message: Updated
Parts:
- removed J1: (no value), SparkFun-Connectors:CONN_06NO_SILK_FEMALE_PTH
- removed SERIEL: (no value), SparkFun-Connectors:CONN_04
- added J2: (no value), SparkFun-Connectors:CONN_05X2PTH
- C3, C4, C5: value (none) -> 100nF
- C6: value (none) -> 1uF; device rcl:C-EUC0603 -> rcl:C-EUC0805
- Q1: value RESONATORSMD -> 16MHz
- R2: value (none) -> 10K
- renumbered Y1 to Q1
Connections:
- removed net N$1: C5.2, SERIEL.1
- new net DTR: C5.2, J2.10
- net CAN_MSG: no longer J1.6
- net CS_CAN: now also J2.5; no longer J1.5
- net GND: now also J2.6, J2.8; no longer J1.1, SERIEL.4
- net MISO: now also J2.3; no longer J1.2
- net MOSI: now also J2.1; no longer J1.3
- net RXD: now also J2.7; no longer SERIEL.2
- net SCK: now also J2.2; no longer J1.4
- net TXD: now also J2.9; no longer SERIEL.3
